File: cc-19-badge.kicad_sch (KiCad schematic)
At the start: 1 part

Commit message: updates
Parts:
- removed U?: ATtiny84A-P, Package_DIP:DIP-14_W7.62mm, symbol MCU_Microchip_ATtiny:ATtiny84A-P
- added U?: ATtiny84A-P, Package_DIP:DIP-14_W7.62mm, symbol MCU_Microchip_ATtiny:ATtiny84A-P
Connections:
- new net +3.3V: U?.1 (VCC)
- new net GND: U?.14 (GND)
Changed lines of the file:
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@@
 (kicad_sch (version 20211123) (generator eeschema)
   (paper "A4")
-  (symbol (lib_id "MCU_Microchip_ATtiny:ATtiny84A-P") (at 90.17 107.95 0) (unit 1)
+  (wire (pts (xy 124.46 119.38) (xy 124.46 121.92))
+    (stroke (width 0) (type default) (color 0 0 0 0))
+  )
+  (wire (pts (xy 124.46 69.85) (xy 124.46 73.66))
+    (stroke (width 0) (type default) (color 0 0 0 0))
+  )
+  (symbol (lib_id "power:+3.3V") (at 124.46 69.85 0) (unit 1)
     (in_bom yes) (on_board yes) (fields_autoplaced)
-    (property "Reference" "U?" (id 0) (at 76.7081 107.1153 0)
+    (property "Reference" "#PWR0102" (id 0) (at 124.46 73.66 0)
+      (effects (font (size 1.27 1.27)) hide)
+    )
+    (property "Value" "+3.3V" (id 1) (at 124.46 66.2742 0))
+    (property "Footprint" "" (id 2) (at 124.46 69.85 0)
+      (effects (font (size 1.27 1.27)) hide)
+    )
+    (property "Datasheet" "" (id 3) (at 124.46 69.85 0)
+      (effects (font (size 1.27 1.27)) hide)
+    )
+    (pin "1")
+  )
+  (symbol (lib_id "power:GND") (at 124.46 121.92 0) (unit 1)
+    (in_bom yes) (on_board yes) (fields_autoplaced)
+    (property "Reference" "#PWR0101" (id 0) (at 124.46 128.27 0)
+      (effects (font (size 1.27 1.27)) hide)
+    )
+    (property "Value" "GND" (id 1) (at 124.46 126.3634 0))
+    (property "Footprint" "" (id 2) (at 124.46 121.92 0)
+      (effects (font (size 1.27 1.27)) hide)
+    )
+    (property "Datasheet" "" (id 3) (at 124.46 121.92 0)
+      (effects (font (size 1.27 1.27)) hide)
+    )
+    (pin "1")
+  )
+  (symbol (lib_id "MCU_Microchip_ATtiny:ATtiny84A-P") (at 124.46 96.52 0) (unit 1)
+    (in_bom yes) (on_board yes) (fields_autoplaced)
+    (property "Reference" "U?" (id 0) (at 110.9981 95.6853 0)
       (effects (font (size 1.27 1.27)) (justify right))
     )
-    (property "Value" "ATtiny84A-P" (id 1) (at 76.7081 109.6522 0)
+    (property "Value" "ATtiny84A-P" (id 1) (at 110.9981 98.2222 0)
       (effects (font (size 1.27 1.27)) (justify right))
     )
-    (property "Footprint" "Package_DIP:DIP-14_W7.62mm" (id 2) (at 90.17 107.95 0)
+    (property "Footprint" "Package_DIP:DIP-14_W7.62mm" (id 2) (at 124.46 96.52 0)
       (effects (font (size 1.27 1.27) italic) hide)
     )
-    (property "Datasheet" "http://ww1.microchip.com/downloads/en/DeviceDoc/doc8183.pdf" (id 3) (at 90.17 107.95 0)
+    (property "Datasheet" "http://ww1.microchip.com/downloads/en/DeviceDoc/doc8183.pdf" (id 3) (at 124.46 96.52 0)
       (effects (font (size 1.27 1.27)) hide)
     )
@@
   )
   (symbol_instances
-    (path "/c53d2f4d-cfa3-4e34-aa9d-268fb6765344"
+    (path "/28701a8b-e9e9-4466-8fbd-2ff8d8c7af4f"
+      (reference "#PWR0101") (unit 1) (value "GND") (footprint "")
+    )
+    (path "/03b8bb26-888a-4324-a542-2f053d7430d1"
+      (reference "#PWR0102") (unit 1) (value "+3.3V") (footprint "")
+    )
+    (path "/b2e1ea54-795e-4622-b6af-e8674d527d3d"
       (reference "U?") (unit 1) (value "ATtiny84A-P") (footprint "Package_DIP:DIP-14_W7.62mm")
     )

Commit message: updates
Parts:
- gave numbers to parts that had none: 1
Connections:
- no-connect marks 0 -> 12
Changed lines of the file:
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@@
 (kicad_sch (version 20211123) (generator eeschema)
   (paper "A4")
+  (no_connect (at 139.7 96.52))
+  (no_connect (at 139.7 106.68))
+  (no_connect (at 139.7 81.28))
+  (no_connect (at 139.7 99.06))
+  (no_connect (at 139.7 109.22))
+  (no_connect (at 139.7 104.14))
+  (no_connect (at 139.7 91.44))
+  (no_connect (at 139.7 86.36))
+  (no_connect (at 139.7 93.98))
+  (no_connect (at 139.7 88.9))
+  (no_connect (at 139.7 83.82))
+  (no_connect (at 139.7 111.76))
   (wire (pts (xy 124.46 119.38) (xy 124.46 121.92))
     (stroke (width 0) (type default) (color 0 0 0 0))
@@
   (symbol (lib_id "MCU_Microchip_ATtiny:ATtiny84A-P") (at 124.46 96.52 0) (unit 1)
     (in_bom yes) (on_board yes) (fields_autoplaced)
-    (property "Reference" "U?" (id 0) (at 110.9981 95.6853 0)
+    (property "Reference" "U1" (id 0) (at 110.9981 95.6853 0)
       (effects (font (size 1.27 1.27)) (justify right))
     )
@@
     )
     (path "/b2e1ea54-795e-4622-b6af-e8674d527d3d"
-      (reference "U?") (unit 1) (value "ATtiny84A-P") (footprint "Package_DIP:DIP-14_W7.62mm")
+      (reference "U1") (unit 1) (value "ATtiny84A-P") (footprint "Package_DIP:DIP-14_W7.62mm")
     )
   )

Commit message: updates
Parts:
- added S1: OS102011MA1QN1, OS102011MA1QN1, symbol OS102011MA1QN1:OS102011MA1QN1
Connections:
- net +3.3V: now also S1.1; no longer U1.1 (VCC)
- new net: S1.2, U1.1 (VCC)
- no-connect marks 12 -> 13
Changed lines of the file:
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@@
   (no_connect (at 139.7 86.36))
   (no_connect (at 139.7 93.98))
+  (no_connect (at 127 60.96))
   (no_connect (at 139.7 88.9))
   (no_connect (at 139.7 83.82))
   (no_connect (at 139.7 111.76))
+  (wire (pts (xy 114.3 60.96) (xy 121.92 60.96))
+    (stroke (width 0) (type default) (color 0 0 0 0))
+  )
+  (wire (pts (xy 124.46 60.96) (xy 124.46 73.66))
+    (stroke (width 0) (type default) (color 0 0 0 0))
+  )
   (wire (pts (xy 124.46 119.38) (xy 124.46 121.92))
     (stroke (width 0) (type default) (color 0 0 0 0))
   )
-  (wire (pts (xy 124.46 69.85) (xy 124.46 73.66))
-    (stroke (width 0) (type default) (color 0 0 0 0))
-  )
-  (symbol (lib_id "power:+3.3V") (at 124.46 69.85 0) (unit 1)
-    (in_bom yes) (on_board yes) (fields_autoplaced)
-    (property "Reference" "#PWR0102" (id 0) (at 124.46 73.66 0)
+  (symbol (lib_id "power:+3.3V") (at 114.3 60.96 90) (unit 1)
+    (in_bom yes) (on_board yes)
+    (property "Reference" "#PWR0102" (id 0) (at 118.11 60.96 0)
       (effects (font (size 1.27 1.27)) hide)
     )
-    (property "Value" "+3.3V" (id 1) (at 124.46 66.2742 0))
-    (property "Footprint" "" (id 2) (at 124.46 69.85 0)
+    (property "Value" "+3.3V" (id 1) (at 110.7242 60.96 0))
+    (property "Footprint" "" (id 2) (at 114.3 60.96 0)
       (effects (font (size 1.27 1.27)) hide)
     )
-    (property "Datasheet" "" (id 3) (at 124.46 69.85 0)
+    (property "Datasheet" "" (id 3) (at 114.3 60.96 0)
       (effects (font (size 1.27 1.27)) hide)
     )
     (pin "1")
+  )
+  (symbol (lib_id "OS102011MA1QN1:OS102011MA1QN1") (at 121.92 60.96 0) (unit 1)
+    (in_bom yes) (on_board yes) (fields_autoplaced)
+    (property "Reference" "S1" (id 0) (at 130.2512 49.9653 0)
+      (effects (font (size 1.27 1.27)) (justify left))
+    )
+    (property "Value" "OS102011MA1QN1" (id 1) (at 130.2512 52.5022 0)
+      (effects (font (size 1.27 1.27)) (justify left))
+    )
+    (property "Footprint" "OS102011MA1QN1" (id 2) (at 130.81 45.72 0)
+      (effects (font (size 1.27 1.27)) (justify left) hide)
+    )
+    (property "Datasheet" "http://www.ckswitches.com/media/1428/os.pdf" (id 3) (at 130.81 48.26 0)
+      (effects (font (size 1.27 1.27)) (justify left) hide)
+    )
+    (property "Description" "Switch Slide Right Angle SPDT 0.1A 12VDC Through Hole Slide Switch SPDT On-On 0.1 A@ 12 V dc Slide" (id 4) (at 130.81 50.8 0)
+      (effects (font (size 1.27 1.27)) (justify left) hide)
+    )
+    (property "Height" "" (id 5) (at 130.81 53.34 0)
+      (effects (font (size 1.27 1.27)) (justify left) hide)
+    )
+    (property "Mouser Part Number" "611-OS102011MA1QN1" (id 6) (at 130.81 55.88 0)
+      (effects (font (size 1.27 1.27)) (justify left) hide)
+    )
+    (property "Mouser Price/Stock" "https://www.mouser.co.uk/ProductDetail/CK/OS102011MA1QN1?qs=WtljUlYws5R6MUgHcLkz4w%3D%3D" (id 7) (at 130.81 58.42 0)
+      (effects (font (size 1.27 1.27)) (justify left) hide)
+    )
+    (property "Manufacturer_Name" "C & K COMPONENTS" (id 8) (at 130.81 60.96 0)
+      (effects (font (size 1.27 1.27)) (justify left) hide)
+    )
+    (property "Manufacturer_Part_Number" "OS102011MA1QN1" (id 9) (at 130.81 63.5 0)
+      (effects (font (size 1.27 1.27)) (justify left) hide)
+    )
+    (pin "1")
+    (pin "2")
+    (pin "3")
   )
   (symbol (lib_id "power:GND") (at 124.46 121.92 0) (unit 1)
@@
       (reference "#PWR0102") (unit 1) (value "+3.3V") (footprint "")
     )
+    (path "/040f8082-76ef-4eb1-ac5d-3018b40eb874"
+      (reference "S1") (unit 1) (value "OS102011MA1QN1") (footprint "OS102011MA1QN1")
+    )
     (path "/b2e1ea54-795e-4622-b6af-e8674d527d3d"

Commit message: updates
Connections:
- net +3.3V: no longer S1.1
- net at S1.2: no longer U1.1 (VCC)
- new net +BATT: S1.1
Changed lines of the file:
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@@
   (no_connect (at 139.7 83.82))
   (no_connect (at 139.7 111.76))
-  (wire (pts (xy 114.3 60.96) (xy 121.92 60.96))
-    (stroke (width 0) (type default) (color 0 0 0 0))
-  )
-  (wire (pts (xy 124.46 60.96) (xy 124.46 73.66))
+  (wire (pts (xy 113.03 60.96) (xy 121.92 60.96))
     (stroke (width 0) (type default) (color 0 0 0 0))
   )
@@
     (stroke (width 0) (type default) (color 0 0 0 0))
   )
-  (symbol (lib_id "power:+3.3V") (at 114.3 60.96 90) (unit 1)
+  (symbol (lib_id "power:+3.3V") (at 138.43 67.31 90) (unit 1)
     (in_bom yes) (on_board yes)
-    (property "Reference" "#PWR0102" (id 0) (at 118.11 60.96 0)
+    (property "Reference" "#PWR0102" (id 0) (at 142.24 67.31 0)
       (effects (font (size 1.27 1.27)) hide)
     )
-    (property "Value" "+3.3V" (id 1) (at 110.7242 60.96 0))
-    (property "Footprint" "" (id 2) (at 114.3 60.96 0)
+    (property "Value" "+3.3V" (id 1) (at 134.8542 67.31 0))
+    (property "Footprint" "" (id 2) (at 138.43 67.31 0)
       (effects (font (size 1.27 1.27)) hide)
     )
-    (property "Datasheet" "" (id 3) (at 114.3 60.96 0)
+    (property "Datasheet" "" (id 3) (at 138.43 67.31 0)
       (effects (font (size 1.27 1.27)) hide)
     )
@@
     (pin "2")
     (pin "3")
+  )
+  (symbol (lib_id "power:+BATT") (at 113.03 60.96 0) (unit 1)
+    (in_bom yes) (on_board yes) (fields_autoplaced)
+    (property "Reference" "#PWR?" (id 0) (at 113.03 64.77 0)
+      (effects (font (size 1.27 1.27)) hide)
+    )
+    (property "Value" "+BATT" (id 1) (at 113.03 57.3842 0))
+    (property "Footprint" "" (id 2) (at 113.03 60.96 0)
+      (effects (font (size 1.27 1.27)) hide)
+    )
+    (property "Datasheet" "" (id 3) (at 113.03 60.96 0)
+      (effects (font (size 1.27 1.27)) hide)
+    )
+    (pin "1")
   )
   (symbol (lib_id "power:GND") (at 124.46 121.92 0) (unit 1)
@@
       (reference "#PWR0102") (unit 1) (value "+3.3V") (footprint "")
     )
+    (path "/0c6b03c7-6d23-4dac-94ab-629cee18b145"
+      (reference "#PWR?") (unit 1) (value "+BATT") (footprint "")
+    )
     (path "/040f8082-76ef-4eb1-ac5d-3018b40eb874"

Commit message: updates
Connections:
- net +3.3V: now also S1.2, U1.1 (VCC)
Other:
- moved on the sheet: S1
Changed lines of the file:
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@@
   (no_connect (at 139.7 86.36))
   (no_connect (at 139.7 93.98))
-  (no_connect (at 127 60.96))
+  (no_connect (at 50.8 46.99))
   (no_connect (at 139.7 88.9))
   (no_connect (at 139.7 83.82))
   (no_connect (at 139.7 111.76))
-  (wire (pts (xy 113.03 60.96) (xy 121.92 60.96))
+  (wire (pts (xy 124.46 71.12) (xy 124.46 73.66))
+    (stroke (width 0) (type default) (color 0 0 0 0))
+  )
+  (wire (pts (xy 48.26 46.99) (xy 48.26 49.53))
     (stroke (width 0) (type default) (color 0 0 0 0))
   )
@@
     (stroke (width 0) (type default) (color 0 0 0 0))
   )
-  (symbol (lib_id "power:+3.3V") (at 138.43 67.31 90) (unit 1)
+  (wire (pts (xy 41.91 46.99) (xy 45.72 46.99))
+    (stroke (width 0) (type default) (color 0 0 0 0))
+  )
+  (symbol (lib_id "power:+3.3V") (at 48.26 49.53 180) (unit 1)
     (in_bom yes) (on_board yes)
-    (property "Reference" "#PWR0102" (id 0) (at 142.24 67.31 0)
+    (property "Reference" "#PWR0102" (id 0) (at 48.26 45.72 0)
       (effects (font (size 1.27 1.27)) hide)
     )
-    (property "Value" "+3.3V" (id 1) (at 134.8542 67.31 0))
-    (property "Footprint" "" (id 2) (at 138.43 67.31 0)
+    (property "Value" "+3.3V" (id 1) (at 48.26 53.1058 0))
+    (property "Footprint" "" (id 2) (at 48.26 49.53 0)
       (effects (font (size 1.27 1.27)) hide)
     )
-    (property "Datasheet" "" (id 3) (at 138.43 67.31 0)
+    (property "Datasheet" "" (id 3) (at 48.26 49.53 0)
       (effects (font (size 1.27 1.27)) hide)
     )
     (pin "1")
   )
-  (symbol (lib_id "OS102011MA1QN1:OS102011MA1QN1") (at 121.92 60.96 0) (unit 1)
+  (symbol (lib_id "OS102011MA1QN1:OS102011MA1QN1") (at 45.72 46.99 0) (unit 1)
     (in_bom yes) (on_board yes) (fields_autoplaced)
-    (property "Reference" "S1" (id 0) (at 130.2512 49.9653 0)
+    (property "Reference" "S1" (id 0) (at 54.0512 35.9953 0)
       (effects (font (size 1.27 1.27)) (justify left))
     )
-    (property "Value" "OS102011MA1QN1" (id 1) (at 130.2512 52.5022 0)
+    (property "Value" "OS102011MA1QN1" (id 1) (at 54.0512 38.5322 0)
       (effects (font (size 1.27 1.27)) (justify left))
     )
-    (property "Footprint" "OS102011MA1QN1" (id 2) (at 130.81 45.72 0)
+    (property "Footprint" "OS102011MA1QN1" (id 2) (at 54.61 31.75 0)
       (effects (font (size 1.27 1.27)) (justify left) hide)
     )
-    (property "Datasheet" "http://www.ckswitches.com/media/1428/os.pdf" (id 3) (at 130.81 48.26 0)
+    (property "Datasheet" "http://www.ckswitches.com/media/1428/os.pdf" (id 3) (at 54.61 34.29 0)
       (effects (font (size 1.27 1.27)) (justify left) hide)
     )
-    (property "Description" "Switch Slide Right Angle SPDT 0.1A 12VDC Through Hole Slide Switch SPDT On-On 0.1 A@ 12 V dc Slide" (id 4) (at 130.81 50.8 0)
+    (property "Description" "Switch Slide Right Angle SPDT 0.1A 12VDC Through Hole Slide Switch SPDT On-On 0.1 A@ 12 V dc Slide" (id 4) (at 54.61 36.83 0)
       (effects (font (size 1.27 1.27)) (justify left) hide)
     )
-    (property "Height" "" (id 5) (at 130.81 53.34 0)
+    (property "Height" "" (id 5) (at 54.61 39.37 0)
       (effects (font (size 1.27 1.27)) (justify left) hide)
     )
-    (property "Mouser Part Number" "611-OS102011MA1QN1" (id 6) (at 130.81 55.88 0)
+    (property "Mouser Part Number" "611-OS102011MA1QN1" (id 6) (at 54.61 41.91 0)
       (effects (font (size 1.27 1.27)) (justify left) hide)
     )
-    (property "Mouser Price/Stock" "https://www.mouser.co.uk/ProductDetail/CK/OS102011MA1QN1?qs=WtljUlYws5R6MUgHcLkz4w%3D%3D" (id 7) (at 130.81 58.42 0)
+    (property "Mouser Price/Stock" "https://www.mouser.co.uk/ProductDetail/CK/OS102011MA1QN1?qs=WtljUlYws5R6MUgHcLkz4w%3D%3D" (id 7) (at 54.61 44.45 0)
       (effects (font (size 1.27 1.27)) (justify left) hide)
     )
-    (property "Manufacturer_Name" "C & K COMPONENTS" (id 8) (at 130.81 60.96 0)
+    (property "Manufacturer_Name" "C & K COMPONENTS" (id 8) (at 54.61 46.99 0)
       (effects (font (size 1.27 1.27)) (justify left) hide)
     )
-    (property "Manufacturer_Part_Number" "OS102011MA1QN1" (id 9) (at 130.81 63.5 0)
+    (property "Manufacturer_Part_Number" "OS102011MA1QN1" (id 9) (at 54.61 49.53 0)
       (effects (font (size 1.27 1.27)) (justify left) hide)
     )
@@
     (pin "3")
   )
-  (symbol (lib_id "power:+BATT") (at 113.03 60.96 0) (unit 1)
+  (symbol (lib_id "power:+BATT") (at 41.91 46.99 90) (unit 1)
     (in_bom yes) (on_board yes) (fields_autoplaced)
-    (property "Reference" "#PWR?" (id 0) (at 113.03 64.77 0)
+    (property "Reference" "#PWR?" (id 0) (at 45.72 46.99 0)
       (effects (font (size 1.27 1.27)) hide)
     )
-    (property "Value" "+BATT" (id 1) (at 113.03 57.3842 0))
-    (property "Footprint" "" (id 2) (at 113.03 60.96 0)
+    (property "Value" "+BATT" (id 1) (at 38.735 47.4238 90)
+      (effects (font (size 1.27 1.27)) (justify left))
+    )
+    (property "Footprint" "" (id 2) (at 41.91 46.99 0)
       (effects (font (size 1.27 1.27)) hide)
     )
-    (property "Datasheet" "" (id 3) (at 113.03 60.96 0)
+    (property "Datasheet" "" (id 3) (at 41.91 46.99 0)
       (effects (font (size 1.27 1.27)) hide)
     )
@@
     )
     (property "Datasheet" "" (id 3) (at 124.46 121.92 0)
+      (effects (font (size 1.27 1.27)) hide)
+    )
+    (pin "1")
+  )
+  (symbol (lib_id "power:+3.3V") (at 124.46 71.12 0) (unit 1)
+    (in_bom yes) (on_board yes)
+    (property "Reference" "#PWR?" (id 0) (at 124.46 74.93 0)
+      (effects (font (size 1.27 1.27)) hide)
+    )
+    (property "Value" "+3.3V" (id 1) (at 124.46 67.5442 0))
+    (property "Footprint" "" (id 2) (at 124.46 71.12 0)
+      (effects (font (size 1.27 1.27)) hide)
+    )
+    (property "Datasheet" "" (id 3) (at 124.46 71.12 0)
       (effects (font (size 1.27 1.27)) hide)
     )
@@
       (reference "#PWR?") (unit 1) (value "+BATT") (footprint "")
     )
+    (path "/4afe1e1a-d515-4b02-b93d-c7f52adc237c"
+      (reference "#PWR?") (unit 1) (value "+3.3V") (footprint "")
+    )
     (path "/040f8082-76ef-4eb1-ac5d-3018b40eb874"

Commit message: updates
Parts:
- added C1: 860020372001, third-party-schematics:CAPPRD200W52D500H1250, symbol 860020372001:860020372001
- added IC1: ST25DV04KC-IE8S3, third-party-schematics:SOIC127P600X175-8N, symbol ST25DV04KC-IE8S3:ST25DV04KC-IE8S3
- added ISP1: Conn_02x03_Odd_Even, Connector_PinHeader_2.54mm:PinHeader_2x03_P2.54mm_Vertical, symbol Connector_Generic:Conn_02x03_Odd_Even
- S1: footprint OS102011MA1QN1 -> third-party-schematics:OS102011MA1QN1; Mouser Price/Stock https://www.mouser.co.uk/ProductDetail/CK/OS102011MA1QN1?qs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 -> https://www.mouser.com/ProductDetail/CK/OS102011MA1QN1?qs=W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
- U1: Mouser Part Number (none) -> 556-ATTINY84A-PU; Mouser Price/Stock (none) -> https://www.mouser.com/ProductDetail/Microchip-Technology-A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
Connections:
- net +3.3V: now also ISP1.2 (Pin_2)
- net GND: now also C1.2, ISP1.6 (Pin_6)
- net RST: now reaches U1.4 (~{RESET}/PB3)
- net RST: now also C1.1, ISP1.5 (Pin_5)
- net MOSI: now reaches U1.7 (PA6)
- net MOSI: now also ISP1.4 (Pin_4)
- net MISO: now reaches U1.8 (PA5)
- net MISO: now also ISP1.1 (Pin_1)
- net SCK: now reaches U1.9 (PA4)
- net SCK: now also ISP1.3 (Pin_3)
- no-connect marks 13 -> 9
Other:
- moved on the sheet: U1

Commit message: updates
Connections:
- net GND: now also IC1.4 (VSS)
Other:
- moved on the sheet: IC1
Changed lines of the file:
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@@
+    (stroke (width 0) (type default) (color 0 0 0 0))
+  )
+  (wire (pts (xy 157.48 104.14) (xy 161.29 104.14))
     (stroke (width 0) (type default) (color 0 0 0 0))
   )
@@
     (pin "1")
   )
-  (symbol (lib_id "ST25DV04KC-IE8S3:ST25DV04KC-IE8S3") (at 91.44 109.22 0) (unit 1)
-    (in_bom yes) (on_board yes) (fields_autoplaced)
-    (property "Reference" "IC1" (id 0) (at 113.03 103.031 0))
-    (property "Value" "ST25DV04KC-IE8S3" (id 1) (at 113.03 105.5679 0))
-    (property "Footprint" "third-party-schematics:SOIC127P600X175-8N" (id 2) (at 130.81 106.68 0)
-      (effects (font (size 1.27 1.27)) (justify left) hide)
-    )
-    (property "Datasheet" "https://www.st.com/resource/en/datasheet/st25dv04kc.pdf" (id 3) (at 130.81 109.22 0)
-      (effects (font (size 1.27 1.27)) (justify left) hide)
-    )
-    (property "Description" "Dynamic NFC/RFID tag IC with 4-Kbit EEPROM, and fast transfer mode capability" (id 4) (at 130.81 111.76 0)
-      (effects (font (size 1.27 1.27)) (justify left) hide)
-    )
-    (property "Height" "1.75" (id 5) (at 130.81 114.3 0)
-      (effects (font (size 1.27 1.27)) (justify left) hide)
-    )
-    (property "Mouser Part Number" "511-ST25DV04KC-IE8S3" (id 6) (at 130.81 116.84 0)
-      (effects (font (size 1.27 1.27)) (justify left) hide)
-    )
-    (property "Mouser Price/Stock" "https://www.mouser.com/ProductDetail/STMicroelectronics/ST25DV04KC-IE8S3?qs=QNEnbhJQKvbdcU8cigvyiw%3D%3D" (id 7) (at 130.81 119.38 0)
-      (effects (font (size 1.27 1.27)) (justify left) hide)
-    )
-    (property "Manufacturer_Name" "STMicroelectronics" (id 8) (at 130.81 121.92 0)
-      (effects (font (size 1.27 1.27)) (justify left) hide)
-    )
-    (property "Manufacturer_Part_Number" "ST25DV04KC-IE8S3" (id 9) (at 130.81 124.46 0)
+  (symbol (lib_id "ST25DV04KC-IE8S3:ST25DV04KC-IE8S3") (at 157.48 111.76 180) (unit 1)
+    (in_bom yes) (on_board yes) (fields_autoplaced)
+    (property "Reference" "IC1" (id 0) (at 135.89 117.949 0))
+    (property "Value" "ST25DV04KC-IE8S3" (id 1) (at 135.89 115.4121 0))
+    (property "Footprint" "third-party-schematics:SOIC127P600X175-8N" (id 2) (at 118.11 114.3 0)
+      (effects (font (size 1.27 1.27)) (justify left) hide)
+    )
+    (property "Datasheet" "https://www.st.com/resource/en/datasheet/st25dv04kc.pdf" (id 3) (at 118.11 111.76 0)
+      (effects (font (size 1.27 1.27)) (justify left) hide)
+    )
+    (property "Description" "Dynamic NFC/RFID tag IC with 4-Kbit EEPROM, and fast transfer mode capability" (id 4) (at 118.11 109.22 0)
+      (effects (font (size 1.27 1.27)) (justify left) hide)
+    )
+    (property "Height" "1.75" (id 5) (at 118.11 106.68 0)
+      (effects (font (size 1.27 1.27)) (justify left) hide)
+    )
+    (property "Mouser Part Number" "511-ST25DV04KC-IE8S3" (id 6) (at 118.11 104.14 0)
+      (effects (font (size 1.27 1.27)) (justify left) hide)
+    )
+    (property "Mouser Price/Stock" "https://www.mouser.com/ProductDetail/STMicroelectronics/ST25DV04KC-IE8S3?qs=QNEnbhJQKvbdcU8cigvyiw%3D%3D" (id 7) (at 118.11 101.6 0)
+      (effects (font (size 1.27 1.27)) (justify left) hide)
+    )
+    (property "Manufacturer_Name" "STMicroelectronics" (id 8) (at 118.11 99.06 0)
+      (effects (font (size 1.27 1.27)) (justify left) hide)
+    )
+    (property "Manufacturer_Part_Number" "ST25DV04KC-IE8S3" (id 9) (at 118.11 96.52 0)
       (effects (font (size 1.27 1.27)) (justify left) hide)
     )
@@
     (pin "8")
   )
+  (symbol (lib_id "power:GND") (at 161.29 104.14 90) (unit 1)
+    (in_bom yes) (on_board yes) (fields_autoplaced)
+    (property "Reference" "#PWR?" (id 0) (at 167.64 104.14 0)
+      (effects (font (size 1.27 1.27)) hide)
+    )
+    (property "Value" "GND" (id 1) (at 164.4649 103.7062 90)
+      (effects (font (size 1.27 1.27)) (justify right))
+    )
+    (property "Footprint" "" (id 2) (at 161.29 104.14 0)
+      (effects (font (size 1.27 1.27)) hide)
+    )
+    (property "Datasheet" "" (id 3) (at 161.29 104.14 0)
+      (effects (font (size 1.27 1.27)) hide)
+    )
+    (pin "1")
+  )
   (sheet_instances
     (path "/" (page "1"))
@@
       (reference "#PWR0107") (unit 1) (value "GND") (footprint "")
     )
+    (path "/fd677a89-1091-4ab4-a33e-a2b19b35cc7c"
+      (reference "#PWR?") (unit 1) (value "GND") (footprint "")
+    )
     (path "/3428f89c-1922-404b-903f-791e8dab1259"

Commit message: updates
Parts:
- added C1, C2: 100nF, third-party-schematics:K104K15X7RF5TH5, symbol K104K15X7RF5TH5:K104K15X7RF5TH5
- added SCL_PULL, SDA_PULL: R_Small, symbol Device:R_Small
- added S_Debug: OS102011MA1QN1, OS102011MA1QN1, symbol OS102011MA1QN1:OS102011MA1QN1
- C_RST1: renamed from C1; value 860020372001 -> 10uF
Connections:
- net +3.3V: now also C1.1, S_Debug.2
- net GND: now also C1.2, C2.2
- net MOSI: now also IC1.6 (SCL), SCL_PULL.2
- net SCK: now also IC1.5 (SDA), SDA_PULL.2
- net at U1.11 (PA2): now also IC1.7 (GPO_(OPEN_DRAIN))
- net VCC: now reaches IC1.8 (VCC)
- net VCC: now also C2.1, SCL_PULL.1, SDA_PULL.1, S_Debug.1
- no-connect marks 9 -> 8
Other:
- moved on the sheet: C_RST1, ISP1
