File: cc-19-badge.kicad_sch (KiCad schematic)
At the start: 10 parts, among them IC1 ST25DV04KC-IE8S3, U1 ATtiny84A-P

Commit message: updates
Parts:
- renumbered SCL_PULL to SCL_PULL1, SDA_PULL to SDA_PULL1, S_Debug to S_Debug1
Connections:
- net VCC: now also S_Debug1.3; no longer S_Debug1.1
Changed lines of the file:
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@@
+    (stroke (width 0) (type default) (color 0 0 0 0))
+  )
+  (wire (pts (xy 138.43 73.66) (xy 140.97 73.66))
     (stroke (width 0) (type default) (color 0 0 0 0))
   )
@@
     (stroke (width 0) (type default) (color 0 0 0 0))
   )
-  (wire (pts (xy 133.35 73.66) (xy 133.35 74.93))
-    (stroke (width 0) (type default) (color 0 0 0 0))
-  )
   (wire (pts (xy 97.79 101.6) (xy 97.79 106.68))
     (stroke (width 0) (type default) (color 0 0 0 0))
@@
   )
   (wire (pts (xy 40.64 74.93) (xy 46.99 74.93))
+    (stroke (width 0) (type default) (color 0 0 0 0))
+  )
+  (wire (pts (xy 140.97 73.66) (xy 140.97 76.2))
     (stroke (width 0) (type default) (color 0 0 0 0))
   )
@@
   (symbol (lib_id "power:VCC") (at 97.79 93.98 0) (unit 1)
     (in_bom yes) (on_board yes) (fields_autoplaced)
-    (property "Reference" "#PWR?" (id 0) (at 97.79 97.79 0)
+    (property "Reference" "#PWR0113" (id 0) (at 97.79 97.79 0)
       (effects (font (size 1.27 1.27)) hide)
     )
@@
   (symbol (lib_id "power:+3.3V") (at 135.89 77.47 180) (unit 1)
     (in_bom yes) (on_board yes) (fields_autoplaced)
-    (property "Reference" "#PWR?" (id 0) (at 135.89 73.66 0)
+    (property "Reference" "#PWR0115" (id 0) (at 135.89 73.66 0)
       (effects (font (size 1.27 1.27)) hide)
     )
@@
   (symbol (lib_id "Device:R_Small") (at 110.49 99.06 0) (unit 1)
     (in_bom yes) (on_board yes) (fields_autoplaced)
-    (property "Reference" "SDA_PULL" (id 0) (at 111.9886 98.2253 0)
+    (property "Reference" "SDA_PULL1" (id 0) (at 111.9886 98.2253 0)
       (effects (font (size 1.27 1.27)) (justify left))
     )
@@
     (pin "2")
   )
-  (symbol (lib_id "power:VCC") (at 133.35 74.93 180) (unit 1)
-    (in_bom yes) (on_board yes) (fields_autoplaced)
-    (property "Reference" "#PWR?" (id 0) (at 133.35 71.12 0)
-      (effects (font (size 1.27 1.27)) hide)
-    )
-    (property "Value" "VCC" (id 1) (at 133.35 79.3734 0))
-    (property "Footprint" "" (id 2) (at 133.35 74.93 0)
-      (effects (font (size 1.27 1.27)) hide)
-    )
-    (property "Datasheet" "" (id 3) (at 133.35 74.93 0)
+  (symbol (lib_id "power:VCC") (at 140.97 76.2 180) (unit 1)
+    (in_bom yes) (on_board yes) (fields_autoplaced)
+    (property "Reference" "#PWR0114" (id 0) (at 140.97 72.39 0)
+      (effects (font (size 1.27 1.27)) hide)
+    )
+    (property "Value" "VCC" (id 1) (at 140.97 80.6434 0))
+    (property "Footprint" "" (id 2) (at 140.97 76.2 0)
+      (effects (font (size 1.27 1.27)) hide)
+    )
+    (property "Datasheet" "" (id 3) (at 140.97 76.2 0)
       (effects (font (size 1.27 1.27)) hide)
     )
@@
   (symbol (lib_id "power:VCC") (at 110.49 93.98 0) (unit 1)
     (in_bom yes) (on_board yes) (fields_autoplaced)
-    (property "Reference" "#PWR?" (id 0) (at 110.49 97.79 0)
+    (property "Reference" "#PWR0112" (id 0) (at 110.49 97.79 0)
       (effects (font (size 1.27 1.27)) hide)
     )
@@
   (symbol (lib_id "OS102011MA1QN1:OS102011MA1QN1") (at 133.35 73.66 0) (unit 1)
     (in_bom yes) (on_board yes) (fields_autoplaced)
-    (property "Reference" "S_Debug" (id 0) (at 141.6812 62.6653 0)
+    (property "Reference" "S_Debug1" (id 0) (at 141.6812 62.6653 0)
       (effects (font (size 1.27 1.27)) (justify left))
     )
@@
   (symbol (lib_id "power:VCC") (at 104.14 111.76 90) (unit 1)
     (in_bom yes) (on_board yes) (fields_autoplaced)
-    (property "Reference" "#PWR?" (id 0) (at 107.95 111.76 0)
+    (property "Reference" "#PWR0111" (id 0) (at 107.95 111.76 0)
       (effects (font (size 1.27 1.27)) hide)
     )
@@
   (symbol (lib_id "Device:R_Small") (at 97.79 99.06 0) (unit 1)
     (in_bom yes) (on_board yes) (fields_autoplaced)
-    (property "Reference" "SCL_PULL" (id 0) (at 99.2886 98.2253 0)
+    (property "Reference" "SCL_PULL1" (id 0) (at 99.2886 98.2253 0)
       (effects (font (size 1.27 1.27)) (justify left))
     )
@@
       (reference "#PWR0110") (unit 1) (value "GND") (footprint "")
     )
+    (path "/e267f27b-94e3-4a9a-8b62-9198d386eb45"
+      (reference "#PWR0111") (unit 1) (value "VCC") (footprint "")
+    )
+    (path "/82db3d0f-12c9-4fa2-aa63-eeca7811f386"
+      (reference "#PWR0112") (unit 1) (value "VCC") (footprint "")
+    )
     (path "/1462f693-0902-4b4f-8482-4ac353d8fa61"
-      (reference "#PWR?") (unit 1) (value "VCC") (footprint "")
+      (reference "#PWR0113") (unit 1) (value "VCC") (footprint "")
+    )
+    (path "/7f72cddb-89b5-4b67-b37c-45871ea8b9ee"
+      (reference "#PWR0114") (unit 1) (value "VCC") (footprint "")
     )
     (path "/3e675a88-54ef-4c6b-a0f4-f567c9b20907"
-      (reference "#PWR?") (unit 1) (value "+3.3V") (footprint "")
-    )
-    (path "/7f72cddb-89b5-4b67-b37c-45871ea8b9ee"
-      (reference "#PWR?") (unit 1) (value "VCC") (footprint "")
-    )
-    (path "/82db3d0f-12c9-4fa2-aa63-eeca7811f386"
-      (reference "#PWR?") (unit 1) (value "VCC") (footprint "")
-    )
-    (path "/e267f27b-94e3-4a9a-8b62-9198d386eb45"
-      (reference "#PWR?") (unit 1) (value "VCC") (footprint "")
+      (reference "#PWR0115") (unit 1) (value "+3.3V") (footprint "")
     )
     (path "/c03a4c90-e8b8-447d-b181-4e51f2d48d27"
@@
     )
     (path "/ee555d95-01f4-401a-8956-de28b353bf6b"
-      (reference "SCL_PULL") (unit 1) (value "R_Small") (footprint "")
+      (reference "SCL_PULL1") (unit 1) (value "R_Small") (footprint "")
     )
     (path "/695f724e-65a2-4242-9cd3-0e6441e6f89e"
-      (reference "SDA_PULL") (unit 1) (value "R_Small") (footprint "")
+      (reference "SDA_PULL1") (unit 1) (value "R_Small") (footprint "")
     )
     (path "/b88ddc05-f750-4f5b-9c61-c4ee95217dd1"
-      (reference "S_Debug") (unit 1) (value "OS102011MA1QN1") (footprint "OS102011MA1QN1")
+      (reference "S_Debug1") (unit 1) (value "OS102011MA1QN1") (footprint "OS102011MA1QN1")
     )
     (path "/b2e1ea54-795e-4622-b6af-e8674d527d3d"

Commit message: updates
Parts:
- removed S_Debug1: OS102011MA1QN1, OS102011MA1QN1, symbol OS102011MA1QN1:OS102011MA1QN1
Connections:
- net VCC: no longer names the net of C2.1, IC1.8 (VCC)
- net VCC: no longer SCL_PULL1.1, SDA_PULL1.1
Changed lines of the file:
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@@
-    (stroke (width 0) (type default) (color 0 0 0 0))
-  )
-  (wire (pts (xy 138.43 73.66) (xy 140.97 73.66))
     (stroke (width 0) (type default) (color 0 0 0 0))
   )
@@
     (stroke (width 0) (type default) (color 0 0 0 0))
   )
-  (wire (pts (xy 140.97 73.66) (xy 140.97 76.2))
-    (stroke (width 0) (type default) (color 0 0 0 0))
-  )
   (wire (pts (xy 223.52 35.56) (xy 229.87 35.56))
     (stroke (width 0) (type default) (color 0 0 0 0))
@@
   )
   (wire (pts (xy 62.23 96.52) (xy 66.04 96.52))
-    (stroke (width 0) (type default) (color 0 0 0 0))
-  )
-  (wire (pts (xy 135.89 73.66) (xy 135.89 77.47))
     (stroke (width 0) (type default) (color 0 0 0 0))
   )
@@
     (pin "6")
   )
-  (symbol (lib_id "power:VCC") (at 97.79 93.98 0) (unit 1)
-    (in_bom yes) (on_board yes) (fields_autoplaced)
-    (property "Reference" "#PWR0113" (id 0) (at 97.79 97.79 0)
-      (effects (font (size 1.27 1.27)) hide)
-    )
-    (property "Value" "VCC" (id 1) (at 99.187 93.1438 0)
-      (effects (font (size 1.27 1.27)) (justify left))
-    )
-    (property "Footprint" "" (id 2) (at 97.79 93.98 0)
-      (effects (font (size 1.27 1.27)) hide)
-    )
-    (property "Datasheet" "" (id 3) (at 97.79 93.98 0)
-      (effects (font (size 1.27 1.27)) hide)
-    )
-    (pin "1")
-  )
   (symbol (lib_id "power:GND") (at 210.82 44.45 0) (unit 1)
     (in_bom yes) (on_board yes) (fields_autoplaced)
@@
     (pin "1")
     (pin "2")
-  )
-  (symbol (lib_id "power:+3.3V") (at 135.89 77.47 180) (unit 1)
-    (in_bom yes) (on_board yes) (fields_autoplaced)
-    (property "Reference" "#PWR0115" (id 0) (at 135.89 73.66 0)
-      (effects (font (size 1.27 1.27)) hide)
-    )
-    (property "Value" "+3.3V" (id 1) (at 135.89 81.9134 0))
-    (property "Footprint" "" (id 2) (at 135.89 77.47 0)
-      (effects (font (size 1.27 1.27)) hide)
-    )
-    (property "Datasheet" "" (id 3) (at 135.89 77.47 0)
-      (effects (font (size 1.27 1.27)) hide)
-    )
-    (pin "1")
   )
   (symbol (lib_id "power:+3.3V") (at 46.99 73.66 0) (unit 1)
@@
     (pin "1")
     (pin "2")
-  )
-  (symbol (lib_id "power:VCC") (at 140.97 76.2 180) (unit 1)
-    (in_bom yes) (on_board yes) (fields_autoplaced)
-    (property "Reference" "#PWR0114" (id 0) (at 140.97 72.39 0)
-      (effects (font (size 1.27 1.27)) hide)
-    )
-    (property "Value" "VCC" (id 1) (at 140.97 80.6434 0))
-    (property "Footprint" "" (id 2) (at 140.97 76.2 0)
-      (effects (font (size 1.27 1.27)) hide)
-    )
-    (property "Datasheet" "" (id 3) (at 140.97 76.2 0)
-      (effects (font (size 1.27 1.27)) hide)
-    )
-    (pin "1")
-  )
-  (symbol (lib_id "power:VCC") (at 110.49 93.98 0) (unit 1)
-    (in_bom yes) (on_board yes) (fields_autoplaced)
-    (property "Reference" "#PWR0112" (id 0) (at 110.49 97.79 0)
-      (effects (font (size 1.27 1.27)) hide)
-    )
-    (property "Value" "VCC" (id 1) (at 111.887 93.1438 0)
-      (effects (font (size 1.27 1.27)) (justify left))
-    )
-    (property "Footprint" "" (id 2) (at 110.49 93.98 0)
-      (effects (font (size 1.27 1.27)) hide)
-    )
-    (property "Datasheet" "" (id 3) (at 110.49 93.98 0)
-      (effects (font (size 1.27 1.27)) hide)
-    )
-    (pin "1")
   )
   (symbol (lib_id "power:GND") (at 25.4 74.93 270) (unit 1)
@@
     (pin "9")
   )
-  (symbol (lib_id "OS102011MA1QN1:OS102011MA1QN1") (at 133.35 73.66 0) (unit 1)
-    (in_bom yes) (on_board yes) (fields_autoplaced)
-    (property "Reference" "S_Debug1" (id 0) (at 141.6812 62.6653 0)
-      (effects (font (size 1.27 1.27)) (justify left))
-    )
-    (property "Value" "OS102011MA1QN1" (id 1) (at 141.6812 65.2022 0)
-      (effects (font (size 1.27 1.27)) (justify left))
-    )
-    (property "Footprint" "OS102011MA1QN1" (id 2) (at 142.24 58.42 0)
-      (effects (font (size 1.27 1.27)) (justify left) hide)
-    )
-    (property "Datasheet" "http://www.ckswitches.com/media/1428/os.pdf" (id 3) (at 142.24 60.96 0)
-      (effects (font (size 1.27 1.27)) (justify left) hide)
-    )
-    (property "Description" "Switch Slide Right Angle SPDT 0.1A 12VDC Through Hole Slide Switch SPDT On-On 0.1 A@ 12 V dc Slide" (id 4) (at 142.24 63.5 0)
-      (effects (font (size 1.27 1.27)) (justify left) hide)
-    )
-    (property "Height" "" (id 5) (at 142.24 66.04 0)
-      (effects (font (size 1.27 1.27)) (justify left) hide)
-    )
-    (property "Mouser Part Number" "611-OS102011MA1QN1" (id 6) (at 142.24 68.58 0)
-      (effects (font (size 1.27 1.27)) (justify left) hide)
-    )
-    (property "Mouser Price/Stock" "https://www.mouser.co.uk/ProductDetail/CK/OS102011MA1QN1?qs=WtljUlYws5R6MUgHcLkz4w%3D%3D" (id 7) (at 142.24 71.12 0)
-      (effects (font (size 1.27 1.27)) (justify left) hide)
-    )
-    (property "Manufacturer_Name" "C & K COMPONENTS" (id 8) (at 142.24 73.66 0)
-      (effects (font (size 1.27 1.27)) (justify left) hide)
-    )
-    (property "Manufacturer_Part_Number" "OS102011MA1QN1" (id 9) (at 142.24 76.2 0)
-      (effects (font (size 1.27 1.27)) (justify left) hide)
-    )
-    (pin "1")
-    (pin "2")
-    (pin "3")
-  )
   (symbol (lib_id "power:+3.3V") (at 251.46 35.56 270) (unit 1)
     (in_bom yes) (on_board yes)
@@
     (pin "8")
   )
-  (symbol (lib_id "power:VCC") (at 104.14 111.76 90) (unit 1)
-    (in_bom yes) (on_board yes) (fields_autoplaced)
-    (property "Reference" "#PWR0111" (id 0) (at 107.95 111.76 0)
-      (effects (font (size 1.27 1.27)) hide)
-    )
-    (property "Value" "VCC" (id 1) (at 100.965 112.1938 90)
-      (effects (font (size 1.27 1.27)) (justify left))
-    )
-    (property "Footprint" "" (id 2) (at 104.14 111.76 0)
-      (effects (font (size 1.27 1.27)) hide)
-    )
-    (property "Datasheet" "" (id 3) (at 104.14 111.76 0)
-      (effects (font (size 1.27 1.27)) hide)
-    )
-    (pin "1")
-  )
   (symbol (lib_id "Device:R_Small") (at 97.79 99.06 0) (unit 1)
     (in_bom yes) (on_board yes) (fields_autoplaced)
@@
       (reference "#PWR0110") (unit 1) (value "GND") (footprint "")
     )
-    (path "/e267f27b-94e3-4a9a-8b62-9198d386eb45"
-      (reference "#PWR0111") (unit 1) (value "VCC") (footprint "")
-    )
-    (path "/82db3d0f-12c9-4fa2-aa63-eeca7811f386"
-      (reference "#PWR0112") (unit 1) (value "VCC") (footprint "")
-    )
-    (path "/1462f693-0902-4b4f-8482-4ac353d8fa61"
-      (reference "#PWR0113") (unit 1) (value "VCC") (footprint "")
-    )
-    (path "/7f72cddb-89b5-4b67-b37c-45871ea8b9ee"
-      (reference "#PWR0114") (unit 1) (value "VCC") (footprint "")
-    )
-    (path "/3e675a88-54ef-4c6b-a0f4-f567c9b20907"
-      (reference "#PWR0115") (unit 1) (value "+3.3V") (footprint "")
-    )
     (path "/c03a4c90-e8b8-447d-b181-4e51f2d48d27"
       (reference "C1") (unit 1) (value "100nF") (footprint "third-party-schematics:K104K15X7RF5TH5")
@@
       (reference "SDA_PULL1") (unit 1) (value "R_Small") (footprint "")
     )
-    (path "/b88ddc05-f750-4f5b-9c61-c4ee95217dd1"
-      (reference "S_Debug1") (unit 1) (value "OS102011MA1QN1") (footprint "OS102011MA1QN1")
-    )
     (path "/b2e1ea54-795e-4622-b6af-e8674d527d3d"

Commit message: updates
Parts:
- removed C_RST1: 10uF, third-party-schematics:CAPPRD200W52D500H1250, symbol 860020372001:860020372001
- removed ISP1: Conn_02x03_Odd_Even, Connector_PinHeader_2.54mm:PinHeader_2x03_P2.54mm_Vertical, symbol Connector_Generic:Conn_02x03_Odd_Even
- removed SCL_PULL1, SDA_PULL1: R_Small, symbol Device:R_Small
- added R1, R2: R_Small, symbol Device:R_Small
Connections:
- net +3.3V: now also C2.1, IC1.8 (VCC), R1.1, R2.1
- net MISO: no longer names the net of U1.8 (PA5)
- net MOSI renamed SCL
- net SCL: now also U1.9 (PA4), R2.2; no longer U1.7 (PA6)
- net SCK renamed SDA
- net SDA: now also U1.7 (PA6), R1.2; no longer U1.9 (PA4)

Commit message: updates
Parts:
- added J1: Conn_01x06, Connector_PinHeader_2.54mm:PinHeader_1x06_P2.54mm_Vertical, symbol Connector_Generic:Conn_01x06
- added LED1, LED2: LTL-4232, third-party-schematics:LTL4232, symbol LTL-4232:LTL-4232
- added R3, R4: 470Ω, third-party-schematics:CFR-Resistor, symbol Device:R_Small
- R1, R2: footprint (none) -> third-party-schematics:CFR-Resistor
Connections:
- net +3.3V: now also J1.1 (Pin_1)
- net GND: now also J1.6 (Pin_6), LED1.2, LED2.2
- net SCL: now also J1.4 (Pin_4)
- net SDA: now also J1.3 (Pin_3)
- net at U1.11 (PA2): no longer IC1.7 (GPO_(OPEN_DRAIN))
- net at U1.5 (PB2): now also R3.1
- net at U1.6 (PA7): now also R4.1
- net at U1.8 (PA5): now also IC1.7 (GPO_(OPEN_DRAIN))
- new net: LED2.1, R4.2
- new net: LED1.1, R3.2
- no-connect marks 8 -> 5

Commit message: pushing to the correct branc this time
Other:
- moved on the sheet: J1
Changed lines of the file:
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@@
     (stroke (width 0) (type default) (color 0 0 0 0))
   )
-  (wire (pts (xy 109.22 66.04) (xy 114.3 66.04))
-    (stroke (width 0) (type default) (color 0 0 0 0))
-  )
-  (wire (pts (xy 119.38 66.04) (xy 119.38 69.85))
+  (wire (pts (xy 121.92 44.45) (xy 127 44.45))
+    (stroke (width 0) (type default) (color 0 0 0 0))
+  )
+  (wire (pts (xy 132.08 44.45) (xy 132.08 48.26))
     (stroke (width 0) (type default) (color 0 0 0 0))
   )
@@
     (stroke (width 0) (type default) (color 0 0 0 0))
   )
-  (wire (pts (xy 121.92 66.04) (xy 121.92 69.85))
+  (wire (pts (xy 134.62 44.45) (xy 134.62 48.26))
     (stroke (width 0) (type default) (color 0 0 0 0))
   )
@@
     (stroke (width 0) (type default) (color 0 0 0 0))
   )
-  (wire (pts (xy 127 66.04) (xy 133.35 66.04))
+  (wire (pts (xy 139.7 44.45) (xy 146.05 44.45))
     (stroke (width 0) (type default) (color 0 0 0 0))
   )
@@
     (effects (font (size 1.27 1.27)) (justify left bottom))
   )
-  (label "SCL" (at 121.92 69.85 270)
+  (label "SCL" (at 134.62 48.26 270)
     (effects (font (size 1.27 1.27)) (justify right bottom))
   )
@@
     (effects (font (size 1.27 1.27)) (justify left bottom))
   )
-  (label "SDA" (at 119.38 69.85 270)
+  (label "SDA" (at 132.08 48.26 270)
     (effects (font (size 1.27 1.27)) (justify right bottom))
   )
@@
     (pin "1")
   )
-  (symbol (lib_id "Connector_Generic:Conn_01x06") (at 119.38 60.96 90) (unit 1)
-    (in_bom yes) (on_board yes) (fields_autoplaced)
-    (property "Reference" "J1" (id 0) (at 120.65 55.9902 90))
-    (property "Value" "Conn_01x06" (id 1) (at 120.65 58.5271 90))
-    (property "Footprint" "Connector_PinHeader_2.54mm:PinHeader_1x06_P2.54mm_Vertical" (id 2) (at 119.38 60.96 0)
-      (effects (font (size 1.27 1.27)) hide)
-    )
-    (property "Datasheet" "~" (id 3) (at 119.38 60.96 0)
+  (symbol (lib_id "Connector_Generic:Conn_01x06") (at 132.08 39.37 90) (unit 1)
+    (in_bom yes) (on_board yes) (fields_autoplaced)
+    (property "Reference" "J1" (id 0) (at 133.35 34.4002 90))
+    (property "Value" "Conn_01x06" (id 1) (at 133.35 36.9371 90))
+    (property "Footprint" "Connector_PinHeader_2.54mm:PinHeader_1x06_P2.54mm_Vertical" (id 2) (at 132.08 39.37 0)
+      (effects (font (size 1.27 1.27)) hide)
+    )
+    (property "Datasheet" "~" (id 3) (at 132.08 39.37 0)
       (effects (font (size 1.27 1.27)) hide)
     )
@@
     (pin "1")
   )
-  (symbol (lib_id "power:+3.3V") (at 109.22 66.04 90) (unit 1)
-    (in_bom yes) (on_board yes) (fields_autoplaced)
-    (property "Reference" "#PWR0111" (id 0) (at 113.03 66.04 0)
-      (effects (font (size 1.27 1.27)) hide)
-    )
-    (property "Value" "+3.3V" (id 1) (at 106.045 66.4738 90)
-      (effects (font (size 1.27 1.27)) (justify left))
-    )
-    (property "Footprint" "" (id 2) (at 109.22 66.04 0)
-      (effects (font (size 1.27 1.27)) hide)
-    )
-    (property "Datasheet" "" (id 3) (at 109.22 66.04 0)
+  (symbol (lib_id "power:+3.3V") (at 121.92 44.45 90) (unit 1)
+    (in_bom yes) (on_board yes) (fields_autoplaced)
+    (property "Reference" "#PWR0111" (id 0) (at 125.73 44.45 0)
+      (effects (font (size 1.27 1.27)) hide)
+    )
+    (property "Value" "+3.3V" (id 1) (at 118.745 44.8838 90)
+      (effects (font (size 1.27 1.27)) (justify left))
+    )
+    (property "Footprint" "" (id 2) (at 121.92 44.45 0)
+      (effects (font (size 1.27 1.27)) hide)
+    )
+    (property "Datasheet" "" (id 3) (at 121.92 44.45 0)
       (effects (font (size 1.27 1.27)) hide)
     )
@@
     (pin "9")
   )
-  (symbol (lib_id "power:GND") (at 133.35 66.04 90) (unit 1)
-    (in_bom yes) (on_board yes) (fields_autoplaced)
-    (property "Reference" "#PWR0112" (id 0) (at 139.7 66.04 0)
-      (effects (font (size 1.27 1.27)) hide)
-    )
-    (property "Value" "GND" (id 1) (at 136.525 66.4738 90)
-      (effects (font (size 1.27 1.27)) (justify right))
-    )
-    (property "Footprint" "" (id 2) (at 133.35 66.04 0)
-      (effects (font (size 1.27 1.27)) hide)
-    )
-    (property "Datasheet" "" (id 3) (at 133.35 66.04 0)
-      (effects (font (size 1.27 1.27)) hide)
-    )
+  (symbol (lib_id "power:GND") (at 146.05 44.45 90) (unit 1)
+    (in_bom yes) (on_board yes) (fields_autoplaced)
+    (property "Reference" "#PWR0112" (id 0) (at 152.4 44.45 0)
+      (effects (font (size 1.27 1.27)) hide)
+    )
+    (property "Value" "GND" (id 1) (at 149.225 44.8838 90)
+      (effects (font (size 1.27 1.27)) (justify right))
+    )
+    (property "Footprint" "" (id 2) (at 146.05 44.45 0)
+      (effects (font (size 1.27 1.27)) hide)
+    )
+    (property "Datasheet" "" (id 3) (at 146.05 44.45 0)
+      (effects (font (size 1.27 1.27)) hide)
+    )

Commit message: updates
Connections:
- net ANT: now reaches IC1.2 (AC0)
- net ANT: now also IC1.3 (AC1)
Changed lines of the file:
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@@
+    (stroke (width 0) (type default) (color 0 0 0 0))
+  )
+  (wire (pts (xy 157.48 106.68) (xy 160.02 106.68))
     (stroke (width 0) (type default) (color 0 0 0 0))
   )
@@
     (stroke (width 0) (type default) (color 0 0 0 0))
   )
+  (wire (pts (xy 157.48 109.22) (xy 160.02 109.22))
+    (stroke (width 0) (type default) (color 0 0 0 0))
+  )
   (wire (pts (xy 99.06 35.56) (xy 99.06 38.1))
     (stroke (width 0) (type default) (color 0 0 0 0))
@@
     (stroke (width 0) (type default) (color 0 0 0 0))
   )
-  (wire (pts (xy 157.48 104.14) (xy 161.29 104.14))
+  (wire (pts (xy 157.48 104.14) (xy 162.56 104.14))
     (stroke (width 0) (type default) (color 0 0 0 0))
   )
   (wire (pts (xy 139.7 44.45) (xy 146.05 44.45))
     (stroke (width 0) (type default) (color 0 0 0 0))
+  )
+  (label "ANT" (at 160.02 109.22 0)
+    (effects (font (size 1.27 1.27)) (justify left bottom))
   )
   (label "SDA" (at 66.04 99.06 0)
@@
   )
   (label "RST" (at 64.77 114.3 0)
+    (effects (font (size 1.27 1.27)) (justify left bottom))
+  )
+  (label "ANT" (at 160.02 106.68 0)
     (effects (font (size 1.27 1.27)) (justify left bottom))
   )
@@
     (pin "1")
   )
-  (symbol (lib_id "power:GND") (at 161.29 104.14 90) (unit 1)
-    (in_bom yes) (on_board yes) (fields_autoplaced)
-    (property "Reference" "#PWR0109" (id 0) (at 167.64 104.14 0)
-      (effects (font (size 1.27 1.27)) hide)
-    )
-    (property "Value" "GND" (id 1) (at 164.4649 103.7062 90)
-      (effects (font (size 1.27 1.27)) (justify right))
-    )
-    (property "Footprint" "" (id 2) (at 161.29 104.14 0)
-      (effects (font (size 1.27 1.27)) hide)
-    )
-    (property "Datasheet" "" (id 3) (at 161.29 104.14 0)
-      (effects (font (size 1.27 1.27)) hide)
-    )
+  (symbol (lib_id "power:GND") (at 162.56 104.14 90) (unit 1)
+    (in_bom yes) (on_board yes) (fields_autoplaced)
+    (property "Reference" "#PWR0109" (id 0) (at 168.91 104.14 0)
+      (effects (font (size 1.27 1.27)) hide)
+    )
+    (property "Value" "GND" (id 1) (at 165.7349 103.7062 90)
+      (effects (font (size 1.27 1.27)) (justify right))
+    )
+    (property "Footprint" "" (id 2) (at 162.56 104.14 0)
+      (effects (font (size 1.27 1.27)) hide)
+    )
+    (property "Datasheet" "" (id 3) (at 162.56 104.14 0)
+      (effects (font (size 1.27 1.27)) hide)
+    )

Commit message: updates
Connections:
- no-connect marks 5 -> 9
Changed lines of the file:
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@@
   (no_connect (at 62.23 109.22))
   (no_connect (at 62.23 83.82))
+  (no_connect (at 62.23 91.44))
   (no_connect (at 62.23 106.68))
+  (no_connect (at 129.54 44.45))
+  (no_connect (at 137.16 44.45))
   (no_connect (at 50.8 46.99))
+  (no_connect (at 62.23 88.9))
   (wire (pts (xy 83.82 35.56) (xy 83.82 38.1))
     (stroke (width 0) (type default) (color 0 0 0 0))
